File: hardware/right/leptosis-right.kicad_sch (KiCad schematic)
At the start: 91 parts, among them J1 USB_C_Receptacle_USB2.0_14P, J2 Conn_01x02, Q2 2N7002, SW10 SW_Push, SW11 SW_Push, SW12 SW_Push, SW14 SW_Push, SW15 SW_Push, SW16 SW_Push, SW17 SW_Push, SW18 SW_Push, SW2 SW_Push, SW22 SW_Push, SW23 SW_Push, SW24 SW_Push, SW3 SW_Push, SW31 SW_SPDT, SW4 SW_Push, SW5 SW_Push, SW6 SW_Push, SW8 SW_Push, SW9 SW_Push, U1 nRF52840, U2 BQ24075RGT, U3 MAX17048X, Y1 32MHz 12pF, Y2 32.768kHz 12.5pF

Commit message: Finished!
Parts:
- L2, L4: LCSC Part # C1035 -> C86083
Changed lines of the file:
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@@
 			)
 		)
-		(property "LCSC Part #" "C1035 "
+		(property "LCSC Part #" "C86083"
 			(at 142.24 114.3 0)
 			(effects
@@
 			)
 		)
-		(property "LCSC Part #" "C1035 "
+		(property "LCSC Part #" "C86083"
 			(at 139.7 114.3 90)
 			(effects
